Commit message: Added all changes with people detecetion, and docking

File: handirob_description/urdf/handirob_1lds.urdf.xacro (robot description, xacro)
@@ -139,37 +139,10 @@
   </joint>
   <link name="imu_link"/>
-  <joint name="scan_joint_right" type="fixed">
+  <joint name="scan_joint" type="fixed">
     <parent link="base_link"/>
-    <child link="right_scan"/>
+    <child link="base_scan"/>
     <origin xyz="0.101374 -0.157273 0.268" rpy="0 0 ${pi}"/>
   </joint>
-  <link name="right_scan">
-    <visual>
-      <origin xyz="0 0 0" rpy="0 0 0"/>
-      <geometry>
-        <mesh filename="package://handirob_description/meshes/sensors/lds.stl" scale="0.001 0.001 0.001"/>
-      </geometry>
-      <material name="dark"/>
-    </visual>
-    <collision>
-      <origin xyz="0 0 0" rpy="0 0 0"/>
-      <geometry>
-        <cylinder length="0.0315" radius="0.055"/>
-      </geometry>
-    </collision>
-    <inertial>
-      <mass value="0.114" />
-      <origin xyz="0 0 0" />
-      <inertia ixx="0.001" ixy="0.0" ixz="0.0"
-               iyy="0.001" iyz="0.0"
-               izz="0.001" />
-    </inertial>
-  </link>
-  <joint name="scan_joint_left" type="fixed">
-    <parent link="base_link"/>
-    <child link="left_scan"/>
-    <origin xyz="0.101374 0.157273 0.268" rpy="0 0 ${pi}"/>
-  </joint>
-  <link name="left_scan">
+  <link name="base_scan">
     <visual>
       <origin xyz="0 0 0" rpy="0 0 0"/>
