Commit message: added meshes

File: handirob_description/urdf/handirob.urdf.xacro (robot description, xacro)
@@ -1,6 +1,6 @@
 <?xml version="1.0" ?>
 <robot name="handirob" xmlns:xacro="http://ros.org/wiki/xacro">
-  <xacro:include filename="$(find turtlebot3_description)/urdf/common_properties.xacro"/>
-  <xacro:include filename="$(find turtlebot3_description)/urdf/turtlebot3_waffle.gazebo.xacro"/>
+  <xacro:include filename="$(find handirob_description)/urdf/common_properties.xacro"/>
+  <!--xacro:include filename="$(find turtlebot3_description)/urdf/turtlebot3_waffle.gazebo.xacro"/-->
   <xacro:property name="r200_cam_rgb_px" value="0.005"/>
   <xacro:property name="r200_cam_rgb_py" value="0.018"/>
@@ -17,5 +17,5 @@
       <origin xyz="0.175 0 0.0" rpy="0 0 0"/>
       <geometry>
-        <mesh filename="package://turtlebot3_description/meshes/bases/waffle_base.stl" scale="0.001 0.001 0.001"/>
+        <mesh filename="package://handirob_description/meshes/bases/waffle_base.stl" scale="0.001 0.001 0.001"/>
       </geometry>
       <material name="light_black"/>
@@ -45,5 +45,5 @@
       <origin xyz="0 0 0" rpy="1.57 0 0"/>
       <geometry>
-        <mesh filename="package://turtlebot3_description/meshes/wheels/left_tire.stl" scale="0.001 0.001 0.001"/>
+        <mesh filename="package://handirob_description/meshes/wheels/left_tire.stl" scale="0.001 0.001 0.001"/>
       </geometry>
       <material name="dark"/>
@@ -73,5 +73,5 @@
       <origin xyz="0 0 0" rpy="1.57 0 0"/>
       <geometry>
-        <mesh filename="package://turtlebot3_description/meshes/wheels/right_tire.stl" scale="0.001 0.001 0.001"/>
+        <mesh filename="package://handirob_description/meshes/wheels/right_tire.stl" scale="0.001 0.001 0.001"/>
       </geometry>
       <material name="dark"/>
@@ -146,5 +146,5 @@
       <origin xyz="0 0 0" rpy="0 0 0"/>
       <geometry>
-        <mesh filename="package://turtlebot3_description/meshes/sensors/lds.stl" scale="0.001 0.001 0.001"/>
+        <mesh filename="package://handirob_description/meshes/sensors/lds.stl" scale="0.001 0.001 0.001"/>
       </geometry>
       <material name="dark"/>
@@ -173,5 +173,5 @@
      <origin xyz="0 0 0" rpy="1.57 0 1.57"/>
       <geometry>
-       <mesh filename="package://turtlebot3_description/meshes/sensors/r200.dae" />
+       <mesh filename="package://handirob_description/meshes/sensors/r200.dae" />
       </geometry>
     </visual>

Commit message: imu link

File: handirob_description/urdf/handirob.urdf.xacro (robot description, xacro)
@@ -135,5 +135,6 @@
     <parent link="base_link"/>
     <child link="imu_link"/>
-    <origin xyz="-0.295 0.135 0.13" rpy="-1.57 0 0"/>
+    <!--origin xyz="-0.295 0.135 0.13" rpy="-1.57 0 0"/-->
+    <origin xyz="-0.295 0.135 0.13" rpy="0 0 0"/>
   </joint>
   <link name="imu_link"/>

Commit message: added lds node

File: handirob_description/urdf/handirob.urdf.xacro (robot description, xacro)
@@ -2,5 +2,4 @@
 <robot name="handirob" xmlns:xacro="http://ros.org/wiki/xacro">
   <xacro:include filename="$(find handirob_description)/urdf/common_properties.xacro"/>
-  <!--xacro:include filename="~/catkin_ws/src/handirob/handirob_description/urdf/common_properties.xacro"/-->
   <!--xacro:include filename="$(find turtlebot3_description)/urdf/turtlebot3_waffle.gazebo.xacro"/-->
   <xacro:property name="r200_cam_rgb_px" value="0.005"/>
@@ -36,5 +35,5 @@
     </inertial>
   </link>
-  <joint name="wheel_left_joint" type="continuous">
+  <joint name="wheel_left_joint" type="fixed">
     <parent link="base_link"/>
     <child link="wheel_left_link"/>
@@ -64,5 +63,5 @@
       </inertial>
   </link>
-  <joint name="wheel_right_joint" type="continuous">
+  <joint name="wheel_right_joint" type="fixed">
     <parent link="base_link"/>
     <child link="wheel_right_link"/>

Commit message: robot launch

File: handirob_description/urdf/handirob.urdf.xacro (robot description, xacro)
@@ -1,6 +1,5 @@
 <?xml version="1.0" ?>
-<robot name="handirob" xmlns:xacro="http://ros.org/wiki/xacro">
+<robot name="turtlebot3_handirob" xmlns:xacro="http://ros.org/wiki/xacro">
   <xacro:include filename="$(find handirob_description)/urdf/common_properties.xacro"/>
-  <!--xacro:include filename="$(find turtlebot3_description)/urdf/turtlebot3_waffle.gazebo.xacro"/-->
   <xacro:property name="r200_cam_rgb_px" value="0.005"/>
   <xacro:property name="r200_cam_rgb_py" value="0.018"/>
@@ -11,23 +10,23 @@
     <parent link="base_footprint"/>
     <child link="base_link" />
-    <origin xyz="0 0 0.010" rpy="0 0 0"/>
+    <origin xyz="0 0 0" rpy="0 0 0"/>
   </joint>
   <link name="base_link">
     <visual>
-      <origin xyz="0.175 0 0.0" rpy="0 0 0"/>
-      <geometry>
-        <mesh filename="package://handirob_description/meshes/bases/waffle_base.stl" scale="0.001 0.001 0.001"/>
+      <origin xyz="0.2 0 0" rpy="1.57 0 4.71"/>
+      <geometry>
+        <mesh filename="package://handirob_description/meshes/bases/handirob_base_no_caster.stl" scale="0.001 0.001 0.001"/>
       </geometry>
       <material name="light_black"/>
     </visual>
     <collision>
-      <origin xyz="0.0 0 0.035" rpy="0 0 0"/>
-      <geometry>
-        <box size="0.37 0.365 0.282"/>
-      </geometry>
-    </collision>
-    <inertial>
-      <origin xyz="0 0 0" rpy="0 0 0"/>
-      <mass value="1.3729096e+00"/>
+      <origin xyz="-0.185 0 0.10" rpy="0 0 0"/>
+      <geometry>
+        <box size="0.379 0.420 0.242"/>
+      </geometry>
+    </collision>
+    <inertial>
+      <origin xyz="-0.185 0 0.070" rpy="0 0 0"/>
+      <mass value="6.442e-02"/>
       <inertia ixx="8.7002718e-03" ixy="-4.7576583e-05" ixz="1.1160499e-04"
                iyy="8.6195418e-03" iyz="-3.5422299e-06"
@@ -35,27 +34,27 @@
     </inertial>
   </link>
-  <joint name="wheel_left_joint" type="fixed">
+  <joint name="wheel_left_joint" type="continuous">
     <parent link="base_link"/>
     <child link="wheel_left_link"/>
-    <origin xyz="0.0 -0.1825 0.09" rpy="-1.57 0 0"/>
+    <origin xyz="0 0.206 0" rpy="1.57 0 3.14"/>
     <axis xyz="0 0 1"/>
   </joint>
   <link name="wheel_left_link">
     <visual>
-      <origin xyz="0 0 0" rpy="1.57 0 0"/>
-      <geometry>
-        <mesh filename="package://handirob_description/meshes/wheels/left_tire.stl" scale="0.001 0.001 0.001"/>
+      <origin xyz="0 0 0" rpy="-1.57 3.14 0"/>
+      <geometry>
+        <mesh filename="package://handirob_description/meshes/wheels/wheel_only.stl" scale="0.001 0.001 0.001"/>
       </geometry>
       <material name="dark"/>
     </visual>
     <collision>
-      <origin xyz="0 0 0" rpy="0 0 0"/>
-      <geometry>
-        <cylinder length="0.025" radius="0.082"/>
-      </geometry>
-    </collision>
-    <inertial>
-      <origin xyz="0 0 0" />
-      <mass value="2.8498940e-02" />
+      <origin xyz="0 0 0.0125" rpy="0 0 3.14"/>
+      <geometry>
+        <cylinder length="0.025" radius="0.0845"/>
+      </geometry>
+    </collision>
+    <inertial>
+      <origin xyz="0 0 0" />
+      <mass value="0.338959" />
       <inertia ixx="1.1175580e-05" ixy="-4.2369783e-11" ixz="-5.9381719e-09"
                iyy="1.1192413e-05" iyz="-1.4400107e-11"
@@ -63,27 +62,27 @@
       </inertial>
   </link>
-  <joint name="wheel_right_joint" type="fixed">
+  <joint name="wheel_right_joint" type="continuous">
     <parent link="base_link"/>
     <child link="wheel_right_link"/>
-    <origin xyz="0.0 0.1825 0.09" rpy="-1.57 0 0"/>
+    <origin xyz="0 -0.206 0" rpy="1.57 0 3.14"/>
     <axis xyz="0 0 1"/>
   </joint>
   <link name="wheel_right_link">
     <visual>
-      <origin xyz="0 0 0" rpy="1.57 0 0"/>
-      <geometry>
-        <mesh filename="package://handirob_description/meshes/wheels/right_tire.stl" scale="0.001 0.001 0.001"/>
+      <origin xyz="0 0 0" rpy="1.57 3.14 0"/>
+      <geometry>
+        <mesh filename="package://handirob_description/meshes/wheels/wheel_only.stl" scale="0.001 0.001 0.001"/>
       </geometry>
       <material name="dark"/>
     </visual>
     <collision>
-      <origin xyz="0 0 0" rpy="0 0 0"/>
-      <geometry>
-        <cylinder length="0.025" radius="0.0825"/>
-      </geometry>
-    </collision>
-    <inertial>
-      <origin xyz="0 0 0" />
-      <mass value="2.8498940e-02" />
+      <origin xyz="0 0 -0.0125" rpy="0 0 3.14"/>
+      <geometry>
+        <cylinder length="0.025" radius="0.0845"/>
+      </geometry>
+    </collision>
+    <inertial>
+      <origin xyz="0 0 0" />
+      <mass value="0.338959" />
       <inertia ixx="1.1175580e-05" ixy="-4.2369783e-11" ixz="-5.9381719e-09"
                iyy="1.1192413e-05" iyz="-1.4400107e-11"
@@ -94,11 +93,11 @@
     <parent link="base_link"/>
     <child link="caster_back_right_link"/>
-    <origin xyz="-0.325 0.15 0.025" rpy="-1.57 0 0"/>
+    <origin xyz="0.4 -0.21 0" rpy="0 0 0"/>
   </joint>
   <link name="caster_back_right_link">
     <collision>
-      <origin xyz="0 0.001 0" rpy="0 0 0"/>
-      <geometry>
-        <box size="0.05 0.065 0.05"/>
+      <origin xyz="0 0.001 0.025" rpy="0 0 0"/>
+      <geometry>
+        <sphere radius="0.032"/>
       </geometry>
     </collision>
@@ -114,11 +113,14 @@
     <parent link="base_link"/>
     <child link="caster_back_left_link"/>
-    <origin xyz="-0.325 -0.015 0.025" rpy="-1.57 0 0"/>
+    <origin xyz="0.4 0.21 0" rpy="0 0 0"/>
   </joint>
   <link name="caster_back_left_link">
     <collision>
-      <origin xyz="0 0.001 0" rpy="0 0 0"/>
-      <geometry>
-        <box size="0.050 0.065 0.05"/>
+      <origin xyz="0 0.001 0.025" rpy="0 0 0"/>
+      <geometry>
+        <sphere radius="0.032"/>
+    <!--
+        <box size="0.165 0.165 0.110"/>
+    -->
       </geometry>
     </collision>
@@ -134,6 +136,5 @@
     <parent link="base_link"/>
     <child link="imu_link"/>
-    <!--origin xyz="-0.295 0.135 0.13" rpy="-1.57 0 0"/-->
-    <origin xyz="-0.295 0.135 0.13" rpy="0 0 0"/>
+    <origin xyz="0.35 -0.135 0.03" rpy="0 0 0"/>
   </joint>
   <link name="imu_link"/>
@@ -141,5 +142,5 @@
     <parent link="base_link"/>
     <child link="base_scan"/>
-    <origin xyz="-0.26 0 0.265" rpy="0 0 0"/>
+    <origin xyz="0.28 0 0.26" rpy="0 0 0"/>
   </joint>
   <link name="base_scan">
@@ -152,5 +153,5 @@
     </visual>
     <collision>
-      <origin xyz="0.015 0 -0.0065" rpy="0 0 0"/>
+      <origin xyz="0.235 0 -0.0065" rpy="0 0 0"/>
       <geometry>
         <cylinder length="0.0315" radius="0.055"/>
@@ -166,5 +167,5 @@
   </link>
   <joint name="camera_joint" type="fixed">
-    <origin xyz="0.064 -0.065 0.094" rpy="0 0 0"/>
+    <origin xyz="-0.064 -0.065 0.094" rpy="0 0 0"/>
     <parent link="base_link"/>
     <child link="camera_link"/>
@@ -183,12 +184,4 @@
       </geometry>
     </collision>
-    <!-- This inertial field needs doesn't contain reliable data!! -->
-<!--   <inertial>
-      <mass value="0.564" />
-      <origin xyz="0 0 0" />
-      <inertia ixx="0.003881243" ixy="0.0" ixz="0.0"
-               iyy="0.000498940" iyz="0.0"
-               izz="0.003879257" />
-    </inertial>-->
   </link>
   <joint name="camera_rgb_joint" type="fixed">

Commit message: lidar range

File: handirob_description/urdf/handirob.urdf.xacro (robot description, xacro)
@@ -7,12 +7,13 @@
   <xacro:property name="r200_cam_depth_offset" value="0.01"/>
   <link name="base_footprint"/>
+    <origin xyz="-0.370 0 0" rpy="0 0 0"/>
   <joint name="base_joint" type="fixed">
     <parent link="base_footprint"/>
     <child link="base_link" />
-    <origin xyz="0 0 0" rpy="0 0 0"/>
+    <origin xyz="0.18 0 0.04" rpy="0 0 0"/>
   </joint>
   <link name="base_link">
     <visual>
-      <origin xyz="0.2 0 0" rpy="1.57 0 4.71"/>
+      <origin xyz="0 0 -0.04" rpy="1.57 0 -1.57"/>
       <geometry>
         <mesh filename="package://handirob_description/meshes/bases/handirob_base_no_caster.stl" scale="0.001 0.001 0.001"/>
@@ -21,5 +22,5 @@
     </visual>
     <collision>
-      <origin xyz="-0.185 0 0.10" rpy="0 0 0"/>
+      <origin xyz="0 0 0.08" rpy="0 0 0"/>
       <geometry>
         <box size="0.379 0.420 0.242"/>
@@ -37,10 +38,10 @@
     <parent link="base_link"/>
     <child link="wheel_left_link"/>
-    <origin xyz="0 0.206 0" rpy="1.57 0 3.14"/>
-    <axis xyz="0 0 1"/>
+    <origin xyz="-0.18 0.206 -0.02" rpy="0 0 0"/>
+    <axis xyz="0 1 0"/>
   </joint>
   <link name="wheel_left_link">
     <visual>
-      <origin xyz="0 0 0" rpy="-1.57 3.14 0"/>
+      <origin xyz="0 0 0" rpy="0 0 0"/>
       <geometry>
         <mesh filename="package://handirob_description/meshes/wheels/wheel_only.stl" scale="0.001 0.001 0.001"/>
@@ -49,5 +50,5 @@
     </visual>
     <collision>
-      <origin xyz="0 0 0.0125" rpy="0 0 3.14"/>
+      <origin xyz="0 0.0125 0" rpy="1.57 0 0"/>
       <geometry>
         <cylinder length="0.025" radius="0.0845"/>
@@ -65,10 +66,10 @@
     <parent link="base_link"/>
     <child link="wheel_right_link"/>
-    <origin xyz="0 -0.206 0" rpy="1.57 0 3.14"/>
-    <axis xyz="0 0 1"/>
+    <origin xyz="-0.18 -0.206 -0.02" rpy="0 0 0"/>
+    <axis xyz="0 1 0"/>
   </joint>
   <link name="wheel_right_link">
     <visual>
-      <origin xyz="0 0 0" rpy="1.57 3.14 0"/>
+      <origin xyz="0 0 0" rpy="3.14 0 0"/>
       <geometry>
         <mesh filename="package://handirob_description/meshes/wheels/wheel_only.stl" scale="0.001 0.001 0.001"/>
@@ -77,5 +78,5 @@
     </visual>
     <collision>
-      <origin xyz="0 0 -0.0125" rpy="0 0 3.14"/>
+      <origin xyz="0 -0.0125 0" rpy="-1.57 0 0"/>
       <geometry>
         <cylinder length="0.025" radius="0.0845"/>
@@ -93,9 +94,9 @@
     <parent link="base_link"/>
     <child link="caster_back_right_link"/>
-    <origin xyz="0.4 -0.21 0" rpy="0 0 0"/>
+    <origin xyz="0.16 -0.21 -0.07" rpy="0 0 0"/>
   </joint>
   <link name="caster_back_right_link">
     <collision>
-      <origin xyz="0 0.001 0.025" rpy="0 0 0"/>
+      <origin xyz="0 0 0" rpy="0 0 0"/>
       <geometry>
         <sphere radius="0.032"/>
@@ -113,14 +114,11 @@
     <parent link="base_link"/>
     <child link="caster_back_left_link"/>
-    <origin xyz="0.4 0.21 0" rpy="0 0 0"/>
+    <origin xyz="0.16 0.21 -0.07" rpy="0 0 0"/>
   </joint>
   <link name="caster_back_left_link">
     <collision>
-      <origin xyz="0 0.001 0.025" rpy="0 0 0"/>
+      <origin xyz="0 0 0" rpy="0 0 0"/>
       <geometry>
         <sphere radius="0.032"/>
-    <!--
-        <box size="0.165 0.165 0.110"/>
-    -->
       </geometry>
     </collision>
@@ -136,5 +134,5 @@
     <parent link="base_link"/>
     <child link="imu_link"/>
-    <origin xyz="0.35 -0.135 0.03" rpy="0 0 0"/>
+    <origin xyz="0.16 -0.15 0" rpy="0 0 0"/>
   </joint>
   <link name="imu_link"/>
@@ -142,5 +140,5 @@
     <parent link="base_link"/>
     <child link="base_scan"/>
-    <origin xyz="0.28 0 0.26" rpy="0 0 0"/>
+    <origin xyz="0 0 0.26" rpy="0 0 0"/>
   </joint>
   <link name="base_scan">
@@ -153,5 +151,5 @@
     </visual>
     <collision>
-      <origin xyz="0.235 0 -0.0065" rpy="0 0 0"/>
+      <origin xyz="0 0 0" rpy="0 0 0"/>
       <geometry>
         <cylinder length="0.0315" radius="0.055"/>
@@ -167,5 +165,5 @@
   </link>
   <joint name="camera_joint" type="fixed">
-    <origin xyz="-0.064 -0.065 0.094" rpy="0 0 0"/>
+    <origin xyz="0.16 -0.065 0." rpy="0 0 0"/>
     <parent link="base_link"/>
     <child link="camera_link"/>

File: handirob_description/urdf/handirob.urdf_old.xacro (robot description, xacro)
@@ -1,6 +1,5 @@
 <?xml version="1.0" ?>
-<robot name="handirob" xmlns:xacro="http://ros.org/wiki/xacro">
+<robot name="turtlebot3_handirob" xmlns:xacro="http://ros.org/wiki/xacro">
   <xacro:include filename="$(find handirob_description)/urdf/common_properties.xacro"/>
-  <!--xacro:include filename="$(find handirob_description)/urdf/turtlebot3_handirob.gazebo.xacro"/-->
   <xacro:property name="r200_cam_rgb_px" value="0.005"/>
   <xacro:property name="r200_cam_rgb_py" value="0.018"/>
@@ -15,5 +14,5 @@
   <link name="base_link">
     <visual>
-      <origin xyz="-0.185 0 -0.04" rpy="1.57 0 -1.57"/>
+      <origin xyz="0.2 0 0" rpy="1.57 0 4.71"/>
       <geometry>
         <mesh filename="package://handirob_description/meshes/bases/handirob_base_no_caster.stl" scale="0.001 0.001 0.001"/>
@@ -34,13 +33,4 @@
                izz="1.4612727e-02" />
     </inertial>
-<!--
-    <inertial>
-      <origin xyz="0.2065 0 0.070" rpy="0 0 0"/>
-      <mass value="6.442e+00"/>
-      <inertia ixx="2.309e+08" ixy="-1.437e+07" ixz="-3.481e+06"
-               iyy="3.355e+08" iyz="-1.125e+07"
-               izz="2.849e+08" />
-    </inertial>
-    -->
   </link>
   <joint name="wheel_left_joint" type="continuous">
@@ -71,18 +61,9 @@
                izz="2.0712558e-05" />
       </inertial>
-<!--
-    <inertial>
-      <origin xyz="0 0 0" />
-      <mass value="0.338959" />
-      <inertia ixx="8.402E+05" ixy="5.709E-08" ixz=" 0.138"
-               iyy="1.535E+06" iyz="4.123E-10"
-               izz="8.402E+05" />
-      </inertial>
-    -->
   </link>
   <joint name="wheel_right_joint" type="continuous">
     <parent link="base_link"/>
     <child link="wheel_right_link"/>
-    <origin xyz="0.0 -0.206 0" rpy="1.57 0 3.14"/>
+    <origin xyz="0 -0.206 0" rpy="1.57 0 3.14"/>
     <axis xyz="0 0 1"/>
   </joint>
@@ -108,18 +89,9 @@
                izz="2.0712558e-05" />
       </inertial>
-<!--
-    <inertial>
-      <origin xyz="0 0 0" />
-      <mass value="0.338959" />
-      <inertia ixx="8.402E+05" ixy="5.709E-08" ixz=" 0.138"
-               iyy="1.535E+06" iyz="4.123E-10"
-               izz="8.402E+05" />
-      </inertial>
-    -->
   </link>
   <joint name="caster_back_right_joint" type="fixed">
     <parent link="base_link"/>
     <child link="caster_back_right_link"/>
-    <origin xyz="-0.335 -0.21 -0.08" rpy="0 0 0"/>
+    <origin xyz="0.4 -0.21 0" rpy="0 0 0"/>
   </joint>
   <link name="caster_back_right_link">
@@ -141,5 +113,5 @@
     <parent link="base_link"/>
     <child link="caster_back_left_link"/>
-    <origin xyz="-0.335 0.21 -0.08" rpy="0 0 0"/>
+    <origin xyz="0.4 0.21 0" rpy="0 0 0"/>
   </joint>
   <link name="caster_back_left_link">
@@ -148,4 +120,7 @@
       <geometry>
         <sphere radius="0.032"/>
+    <!--
+        <box size="0.165 0.165 0.110"/>
+    -->
       </geometry>
     </collision>
@@ -161,11 +136,11 @@
     <parent link="base_link"/>
     <child link="imu_link"/>
-    <origin xyz="-0.295 0.135 0.13" rpy="0 0 0"/>
+    <origin xyz="0.35 -0.135 0.03" rpy="0 0 0"/>
   </joint>
   <link name="imu_link"/>
-  <joint name="scan_joint_1" type="fixed">
+  <joint name="scan_joint" type="fixed">
     <parent link="base_link"/>
     <child link="base_scan"/>
-    <origin xyz="-0.3 0 0.26" rpy="0 0 0"/>
+    <origin xyz="0.28 0 0.26" rpy="0 0 0"/>
   </joint>
   <link name="base_scan">
@@ -178,5 +153,5 @@
     </visual>
     <collision>
-      <origin xyz="0.015 0 -0.0065" rpy="0 0 0"/>
+      <origin xyz="0.235 0 -0.0065" rpy="0 0 0"/>
       <geometry>
         <cylinder length="0.0315" radius="0.055"/>
@@ -209,12 +184,4 @@
       </geometry>
     </collision>
-    <!-- This inertial field needs doesn't contain reliable data!! -->
-<!--   <inertial>
-      <mass value="0.564" />
-      <origin xyz="0 0 0" />
-      <inertia ixx="0.003881243" ixy="0.0" ixz="0.0"
-               iyy="0.000498940" iyz="0.0"
-               izz="0.003879257" />
-    </inertial>-->
   </link>
   <joint name="camera_rgb_joint" type="fixed">

Commit message: added realsense

File: handirob_description/urdf/handirob.urdf.xacro (robot description, xacro)
@@ -134,5 +134,5 @@
     <parent link="base_link"/>
     <child link="imu_link"/>
-    <origin xyz="0.16 -0.15 0" rpy="0 0 0"/>
+    <origin xyz="0.16 -0.15 0" rpy="0 0 3.1415"/>
   </joint>
   <link name="imu_link"/>

Commit message: removed camera urdf

File: handirob_description/urdf/handirob.urdf.xacro (robot description, xacro)
@@ -183,5 +183,5 @@
     </collision>
   </link>
-  <joint name="camera_rgb_joint" type="fixed">
+  <!--joint name="camera_rgb_joint" type="fixed">
     <origin xyz="${r200_cam_rgb_px} ${r200_cam_rgb_py} ${r200_cam_rgb_pz}" rpy="0 0 0"/>
     <parent link="camera_link"/>
@@ -206,4 +206,4 @@
     <child link="camera_depth_optical_frame"/>
   </joint>
-  <link name="camera_depth_optical_frame"/>
+  <link name="camera_depth_optical_frame"/-->
 </robot>

Commit message: added camera with model

File: handirob_description/urdf/handirob.urdf.xacro (robot description, xacro)
@@ -2,4 +2,5 @@
 <robot name="turtlebot3_handirob" xmlns:xacro="http://ros.org/wiki/xacro">
   <xacro:include filename="$(find handirob_description)/urdf/common_properties.xacro"/>
+  <!--xacro:include filename="$(find realsense2_description)/urdf/_d435.urdf.xacro" /-->
   <xacro:property name="r200_cam_rgb_px" value="0.005"/>
   <xacro:property name="r200_cam_rgb_py" value="0.018"/>
@@ -165,11 +166,13 @@
   </link>
   <joint name="camera_joint" type="fixed">
-    <origin xyz="0.16 -0.065 0." rpy="0 0 0"/>
+    <origin xyz="0.2 0 0.1" rpy="0 0 0"/>
+    <!--origin xyz="0.16 -0.065 0.1" rpy="0 0 0"/-->
     <parent link="base_link"/>
     <child link="camera_link"/>
   </joint>
+<!--origin xyz="0 0 0" rpy="1.57 0 1.57"/-->
   <link name="camera_link">
-    <visual>
-     <origin xyz="0 0 0" rpy="1.57 0 1.57"/>
+    <!--visual>
+     <origin xyz="0 0 0" rpy="0 0 0"/>
       <geometry>
        <mesh filename="package://handirob_description/meshes/sensors/r200.dae" />
@@ -181,5 +184,5 @@
         <box size="0.012 0.132 0.020"/>
       </geometry>
-    </collision>
+    </collision-->
   </link>
   <!--joint name="camera_rgb_joint" type="fixed">
