Commit message: edit robot launch

File: handirob_description/urdf/handirob.urdf.xacro (robot description, xacro)
@@ -1,20 +1,20 @@
 <?xml version="1.0" ?>
-<robot name="turtlebot3_handirob" xmlns:xacro="http://ros.org/wiki/xacro">
+<robot name="handirob" xmlns:xacro="http://ros.org/wiki/xacro">
   <xacro:include filename="$(find handirob_description)/urdf/common_properties.xacro"/>
-  <!--xacro:include filename="$(find realsense2_description)/urdf/_d435.urdf.xacro" /-->
-  <xacro:property name="r200_cam_rgb_px" value="0.005"/>
-  <xacro:property name="r200_cam_rgb_py" value="0.018"/>
-  <xacro:property name="r200_cam_rgb_pz" value="0.013"/>
-  <xacro:property name="r200_cam_depth_offset" value="0.01"/>
+  <xacro:include filename="$(find realsense2_description)/urdf/_d435.urdf.xacro" />
+  <xacro:property name="base_offset_x" value="0.20625"/>
+  <xacro:property name="base_offset_y" value="0.206"/>
+  <xacro:property name="base_offset_z" value="0.041"/>
+  <xacro:property name="pi" value="3.14159"/>
   <link name="base_footprint"/>
-    <origin xyz="-0.370 0 0" rpy="0 0 0"/>
+    <origin xyz="0 0 0" rpy="0 0 0"/>
   <joint name="base_joint" type="fixed">
     <parent link="base_footprint"/>
     <child link="base_link" />
-    <origin xyz="0.18 0 0.04" rpy="0 0 0"/>
+    <origin xyz="-${base_offset_x} 0 -0.041" rpy="0 0 0"/>
   </joint>
   <link name="base_link">
     <visual>
-      <origin xyz="0 0 -0.04" rpy="1.57 0 -1.57"/>
+      <origin xyz="0 0 0" rpy="${pi}/2 0 -${pi}/2"/>
       <geometry>
         <mesh filename="package://handirob_description/meshes/bases/handirob_base_no_caster.stl" scale="0.001 0.001 0.001"/>
@@ -39,5 +39,5 @@
     <parent link="base_link"/>
     <child link="wheel_left_link"/>
-    <origin xyz="-0.18 0.206 -0.02" rpy="0 0 0"/>
+    <origin xyz="${base_offset_x} ${base_offset_y} ${base_offset_z}" rpy="0 0 0"/>
     <axis xyz="0 1 0"/>
   </joint>
@@ -51,5 +51,5 @@
     </visual>
     <collision>
-      <origin xyz="0 0.0125 0" rpy="1.57 0 0"/>
+      <origin xyz="0 0.0125 0" rpy="${pi}/2 0 0"/>
       <geometry>
         <cylinder length="0.025" radius="0.0845"/>
@@ -67,10 +67,10 @@
     <parent link="base_link"/>
     <child link="wheel_right_link"/>
-    <origin xyz="-0.18 -0.206 -0.02" rpy="0 0 0"/>
+    <origin xyz="${base_offset_x} -${base_offset_y} ${base_offset_z}" rpy="0 0 0"/>
     <axis xyz="0 1 0"/>
   </joint>
   <link name="wheel_right_link">
     <visual>
-      <origin xyz="0 0 0" rpy="3.14 0 0"/>
+      <origin xyz="0 0 0" rpy="${pi} 0 0"/>
       <geometry>
         <mesh filename="package://handirob_description/meshes/wheels/wheel_only.stl" scale="0.001 0.001 0.001"/>
@@ -79,5 +79,5 @@
     </visual>
     <collision>
-      <origin xyz="0 -0.0125 0" rpy="-1.57 0 0"/>
+      <origin xyz="0 -0.0125 0" rpy="-${pi}/2 0 0"/>
       <geometry>
         <cylinder length="0.025" radius="0.0845"/>
@@ -95,5 +95,5 @@
     <parent link="base_link"/>
     <child link="caster_back_right_link"/>
-    <origin xyz="0.16 -0.21 -0.07" rpy="0 0 0"/>
+    <origin xyz="-0.2 -0.21 0" rpy="0 0 0"/>
   </joint>
   <link name="caster_back_right_link">
@@ -115,5 +115,5 @@
     <parent link="base_link"/>
     <child link="caster_back_left_link"/>
-    <origin xyz="0.16 0.21 -0.07" rpy="0 0 0"/>
+    <origin xyz="-0.2 0.21 0" rpy="0 0 0"/>
   </joint>
   <link name="caster_back_left_link">
@@ -135,5 +135,5 @@
     <parent link="base_link"/>
     <child link="imu_link"/>
-    <origin xyz="0.16 -0.15 0" rpy="0 0 3.1415"/>
+    <origin xyz="0.185 -0.048 0.145" rpy="0 0 ${pi}"/>
   </joint>
   <link name="imu_link"/>
@@ -141,5 +141,5 @@
     <parent link="base_link"/>
     <child link="base_scan"/>
-    <origin xyz="0 0 0.26" rpy="0 0 0"/>
+    <origin xyz="0.101374 0.157273 0.268" rpy="0 0 ${pi}"/>
   </joint>
   <link name="base_scan">
@@ -165,48 +165,6 @@
     </inertial>
   </link>
-  <joint name="camera_joint" type="fixed">
-    <origin xyz="0.2 0 0.1" rpy="0 0 0"/>
-    <!--origin xyz="0.16 -0.065 0.1" rpy="0 0 0"/-->
-    <parent link="base_link"/>
-    <child link="camera_link"/>
-  </joint>
-<!--origin xyz="0 0 0" rpy="1.57 0 1.57"/-->
-  <link name="camera_link">
-    <!--visual>
-     <origin xyz="0 0 0" rpy="0 0 0"/>
-      <geometry>
-       <mesh filename="package://handirob_description/meshes/sensors/r200.dae" />
-      </geometry>
-    </visual>
-    <collision>
-      <origin xyz="0.003 0.065 0.007" rpy="0 0 0"/>
-      <geometry>
-        <box size="0.012 0.132 0.020"/>
-      </geometry>
-    </collision-->
-  </link>
-  <!--joint name="camera_rgb_joint" type="fixed">
-    <origin xyz="${r200_cam_rgb_px} ${r200_cam_rgb_py} ${r200_cam_rgb_pz}" rpy="0 0 0"/>
-    <parent link="camera_link"/>
-    <child link="camera_rgb_frame"/>
-  </joint>
-  <link name="camera_rgb_frame"/>
-  <joint name="camera_rgb_optical_joint" type="fixed">
-    <origin xyz="0 0 0" rpy="-1.57 0 -1.57"/>
-    <parent link="camera_rgb_frame"/>
-    <child link="camera_rgb_optical_frame"/>
-  </joint>
-  <link name="camera_rgb_optical_frame"/>
-  <joint name="camera_depth_joint" type="fixed">
-    <origin xyz="${r200_cam_rgb_px} ${r200_cam_rgb_py + r200_cam_depth_offset} ${r200_cam_rgb_pz}" rpy="0 0 0"/>
-    <parent link="camera_link"/>
-    <child link="camera_depth_frame"/>
-  </joint>
-  <link name="camera_depth_frame"/>
-  <joint name="camera_depth_optical_joint" type="fixed">
-    <origin xyz="0 0 0" rpy="-1.57 0 -1.57"/>
-    <parent link="camera_depth_frame"/>
-    <child link="camera_depth_optical_frame"/>
-  </joint>
-  <link name="camera_depth_optical_frame"/-->
+<xacro:sensor_d435 parent="base_link" use_nominal_extrinsics="false" add_plug="false" use_mesh="true">
+  <origin xyz="0.215 0.016 0.18" rpy="0 0 0"/>
+</xacro:sensor_d435>
 </robot>

File: handirob_description/urdf/handirob_v1.urdf.xacro (robot description, xacro)
@@ -2,4 +2,5 @@
 <robot name="turtlebot3_handirob" xmlns:xacro="http://ros.org/wiki/xacro">
   <xacro:include filename="$(find handirob_description)/urdf/common_properties.xacro"/>
+  <xacro:include filename="$(find realsense2_description)/urdf/_d435.urdf.xacro" />
   <xacro:property name="r200_cam_rgb_px" value="0.005"/>
   <xacro:property name="r200_cam_rgb_py" value="0.018"/>
@@ -7,12 +8,13 @@
   <xacro:property name="r200_cam_depth_offset" value="0.01"/>
   <link name="base_footprint"/>
+    <origin xyz="-0.370 0 0" rpy="0 0 0"/>
   <joint name="base_joint" type="fixed">
     <parent link="base_footprint"/>
     <child link="base_link" />
-    <origin xyz="0 0 0" rpy="0 0 0"/>
+    <origin xyz="0.18 0 0.04" rpy="0 0 0"/>
   </joint>
   <link name="base_link">
     <visual>
-      <origin xyz="0.2 0 0" rpy="1.57 0 4.71"/>
+      <origin xyz="0 0 -0.04" rpy="1.57 0 -1.57"/>
       <geometry>
         <mesh filename="package://handirob_description/meshes/bases/handirob_base_no_caster.stl" scale="0.001 0.001 0.001"/>
@@ -21,5 +23,5 @@
     </visual>
     <collision>
-      <origin xyz="-0.185 0 0.10" rpy="0 0 0"/>
+      <origin xyz="0 0 0.08" rpy="0 0 0"/>
       <geometry>
         <box size="0.379 0.420 0.242"/>
@@ -37,10 +39,10 @@
     <parent link="base_link"/>
     <child link="wheel_left_link"/>
-    <origin xyz="0 0.206 0" rpy="1.57 0 3.14"/>
-    <axis xyz="0 0 1"/>
+    <origin xyz="-0.18 0.206 -0.02" rpy="0 0 0"/>
+    <axis xyz="0 1 0"/>
   </joint>
   <link name="wheel_left_link">
     <visual>
-      <origin xyz="0 0 0" rpy="-1.57 3.14 0"/>
+      <origin xyz="0 0 0" rpy="0 0 0"/>
       <geometry>
         <mesh filename="package://handirob_description/meshes/wheels/wheel_only.stl" scale="0.001 0.001 0.001"/>
@@ -49,5 +51,5 @@
     </visual>
     <collision>
-      <origin xyz="0 0 0.0125" rpy="0 0 3.14"/>
+      <origin xyz="0 0.0125 0" rpy="1.57 0 0"/>
       <geometry>
         <cylinder length="0.025" radius="0.0845"/>
@@ -65,10 +67,10 @@
     <parent link="base_link"/>
     <child link="wheel_right_link"/>
-    <origin xyz="0 -0.206 0" rpy="1.57 0 3.14"/>
-    <axis xyz="0 0 1"/>
+    <origin xyz="-0.18 -0.206 -0.02" rpy="0 0 0"/>
+    <axis xyz="0 1 0"/>
   </joint>
   <link name="wheel_right_link">
     <visual>
-      <origin xyz="0 0 0" rpy="1.57 3.14 0"/>
+      <origin xyz="0 0 0" rpy="3.14 0 0"/>
       <geometry>
         <mesh filename="package://handirob_description/meshes/wheels/wheel_only.stl" scale="0.001 0.001 0.001"/>
@@ -77,5 +79,5 @@
     </visual>
     <collision>
-      <origin xyz="0 0 -0.0125" rpy="0 0 3.14"/>
+      <origin xyz="0 -0.0125 0" rpy="-1.57 0 0"/>
       <geometry>
         <cylinder length="0.025" radius="0.0845"/>
@@ -93,9 +95,9 @@
     <parent link="base_link"/>
     <child link="caster_back_right_link"/>
-    <origin xyz="0.4 -0.21 0" rpy="0 0 0"/>
+    <origin xyz="0.16 -0.21 -0.07" rpy="0 0 0"/>
   </joint>
   <link name="caster_back_right_link">
     <collision>
-      <origin xyz="0 0.001 0.025" rpy="0 0 0"/>
+      <origin xyz="0 0 0" rpy="0 0 0"/>
       <geometry>
         <sphere radius="0.032"/>
@@ -113,14 +115,11 @@
     <parent link="base_link"/>
     <child link="caster_back_left_link"/>
-    <origin xyz="0.4 0.21 0" rpy="0 0 0"/>
+    <origin xyz="0.16 0.21 -0.07" rpy="0 0 0"/>
   </joint>
   <link name="caster_back_left_link">
     <collision>
-      <origin xyz="0 0.001 0.025" rpy="0 0 0"/>
+      <origin xyz="0 0 0" rpy="0 0 0"/>
       <geometry>
         <sphere radius="0.032"/>
-    <!--
-        <box size="0.165 0.165 0.110"/>
-    -->
       </geometry>
     </collision>
@@ -136,5 +135,5 @@
     <parent link="base_link"/>
     <child link="imu_link"/>
-    <origin xyz="0.35 -0.135 0.03" rpy="0 0 0"/>
+    <origin xyz="0.16 -0.15 0" rpy="0 0 3.1415"/>
   </joint>
   <link name="imu_link"/>
@@ -142,5 +141,5 @@
     <parent link="base_link"/>
     <child link="base_scan"/>
-    <origin xyz="0.28 0 0.26" rpy="0 0 0"/>
+    <origin xyz="0 0 0.26" rpy="0 0 0"/>
   </joint>
   <link name="base_scan">
@@ -153,5 +152,5 @@
     </visual>
     <collision>
-      <origin xyz="0.235 0 -0.0065" rpy="0 0 0"/>
+      <origin xyz="0 0 0" rpy="0 0 0"/>
       <geometry>
         <cylinder length="0.0315" radius="0.055"/>
@@ -166,12 +165,19 @@
     </inertial>
   </link>
-  <joint name="camera_joint" type="fixed">
-    <origin xyz="-0.064 -0.065 0.094" rpy="0 0 0"/>
+    <!--origin xyz="0.16 -0.065 0.1" rpy="0 0 0"/-->
+  <!--joint name="camera_joint" type="fixed">
+    <origin xyz="0.2 0 0.1" rpy="0 0 0"/>
     <parent link="base_link"/>
     <child link="camera_link"/>
-  </joint>
-  <link name="camera_link">
-    <visual>
-     <origin xyz="0 0 0" rpy="1.57 0 1.57"/>
+  </joint-->
+<!--link name="camera_link"/-->
+<xacro:sensor_d435 parent="base_link" use_nominal_extrinsics="false" add_plug="false" use_mesh="true">
+  <origin xyz="0.2 0 0.1" rpy="0 0 0"/>
+</xacro:sensor_d435>
+<!--/xacro:sensor_d435-->
+<!--origin xyz="0 0 0" rpy="1.57 0 1.57"/-->
+  <!--link name="camera_link"-->
+    <!--visual>
+     <origin xyz="0 0 0" rpy="0 0 0"/>
       <geometry>
        <mesh filename="package://handirob_description/meshes/sensors/r200.dae" />
@@ -183,7 +189,7 @@
         <box size="0.012 0.132 0.020"/>
       </geometry>
-    </collision>
-  </link>
-  <joint name="camera_rgb_joint" type="fixed">
+    </collision-->
+  <!--/link-->
+  <!--joint name="camera_rgb_joint" type="fixed">
     <origin xyz="${r200_cam_rgb_px} ${r200_cam_rgb_py} ${r200_cam_rgb_pz}" rpy="0 0 0"/>
     <parent link="camera_link"/>
@@ -208,4 +214,4 @@
     <child link="camera_depth_optical_frame"/>
   </joint>
-  <link name="camera_depth_optical_frame"/>
+  <link name="camera_depth_optical_frame"/-->
 </robot>

Commit message: added realsense

File: handirob_description/urdf/handirob.urdf.xacro (robot description, xacro)
@@ -6,5 +6,6 @@
   <xacro:property name="base_offset_y" value="0.206"/>
   <xacro:property name="base_offset_z" value="0.041"/>
-  <xacro:property name="pi" value="3.14159"/>
+  <!--xacro:property name="pi" value="3.14159"/-->
+  <xacro:property name="pi_half" value="1.570795"/>
   <link name="base_footprint"/>
     <origin xyz="0 0 0" rpy="0 0 0"/>
@@ -16,5 +17,5 @@
   <link name="base_link">
     <visual>
-      <origin xyz="0 0 0" rpy="${pi}/2 0 -${pi}/2"/>
+      <origin xyz="0 0 0" rpy="${pi_half} 0 -${pi_half}"/>
       <geometry>
         <mesh filename="package://handirob_description/meshes/bases/handirob_base_no_caster.stl" scale="0.001 0.001 0.001"/>
@@ -51,5 +52,5 @@
     </visual>
     <collision>
-      <origin xyz="0 0.0125 0" rpy="${pi}/2 0 0"/>
+      <origin xyz="0 0.0125 0" rpy="${pi_half} 0 0"/>
       <geometry>
         <cylinder length="0.025" radius="0.0845"/>
@@ -79,5 +80,5 @@
     </visual>
     <collision>
-      <origin xyz="0 -0.0125 0" rpy="-${pi}/2 0 0"/>
+      <origin xyz="0 -0.0125 0" rpy="-${pi_half} 0 0"/>
       <geometry>
         <cylinder length="0.025" radius="0.0845"/>
@@ -141,5 +142,5 @@
     <parent link="base_link"/>
     <child link="base_scan"/>
-    <origin xyz="0.101374 0.157273 0.268" rpy="0 0 ${pi}"/>
+    <origin xyz="0.101374 -0.157273 0.268" rpy="0 0 ${pi}"/>
   </joint>
   <link name="base_scan">

Commit message: Added openCR arudino files and other modifications

File: handirob_description/urdf/handirob.urdf.xacro (robot description, xacro)
@@ -194,5 +194,5 @@
   </link>
 <xacro:sensor_d435 parent="base_link" use_nominal_extrinsics="false" add_plug="false" use_mesh="true">
-  <origin xyz="0.215 0.016 0.18" rpy="0 0 0"/>
+  <origin xyz="0.215 0.016 0.18" rpy="0 -0.6 0"/>
 </xacro:sensor_d435>
 </robot>
