Commit message: Add all dingle dangle

File: handirob_description/urdf/handirob.urdf.xacro (robot description, xacro)
@@ -6,126 +6,139 @@
   <xacro:property name="base_offset_y" value="0.206"/>
   <xacro:property name="base_offset_z" value="0.041"/>
-  <!--xacro:property name="pi" value="3.14159"/-->
-  <xacro:property name="pi_half" value="1.570795"/>
-  <link name="base_footprint"/>
+  <xacro:property name="pi" value="3.1415926535897931"/>
+  <xacro:property name="pi_half" value="${pi/2}"/>
+  <link name="base_link"/>
     <origin xyz="0 0 0" rpy="0 0 0"/>
   <joint name="base_joint" type="fixed">
-    <parent link="base_footprint"/>
-    <child link="base_link" />
-    <origin xyz="-${base_offset_x} 0 -0.041" rpy="0 0 0"/>
-  </joint>
-  <link name="base_link">
-    <visual>
-      <origin xyz="0 0 0" rpy="${pi_half} 0 -${pi_half}"/>
-      <geometry>
-        <mesh filename="package://handirob_description/meshes/bases/handirob_base_no_caster.stl" scale="0.001 0.001 0.001"/>
+    <parent link="base_link"/>
+    <child link="differential_link" />
+    <!--
+    <origin xyz="0 0 -0.041" rpy="0 0 0"/>
+    -->
+    <origin xyz="0 0 0" rpy="0 0 0"/>
+  </joint>
+  <link name="differential_link">
+    <visual>
+      <origin xyz="0 0 -0.041" rpy="${pi_half}  0 -${pi_half}"/>
+      <geometry>
+        <mesh filename="package://handirob_description/meshes/bases/handirob_Shell.stl" scale="0.001 0.001 0.001"/>
       </geometry>
       <material name="light_black"/>
     </visual>
     <collision>
-      <origin xyz="0 0 0.08" rpy="0 0 0"/>
-      <geometry>
-        <box size="0.379 0.420 0.242"/>
-      </geometry>
-    </collision>
-    <inertial>
-      <origin xyz="-0.185 0 0.070" rpy="0 0 0"/>
-      <mass value="6.442e-02"/>
+      <origin xyz="0 0 0.09" rpy="0 0 0"/>
+      <geometry>
+        <box size="0.645 0.53 0.262"/>
+      </geometry>
+    </collision>
+    <inertial>
+      <origin xyz="0.2 0 0" rpy="0 0 0"/>
+      <mass value="7"/>
+    <inertia ixx="0.001" ixy="0.00" ixz="0.01"
+               iyy="0.001" iyz="0.00"
+               izz="0.001" />
+    </inertial>
+    <!--
+      <inertia ixx="0.044" ixy="0.00" ixz="0.04"
+               iyy="0.025" iyz="0.00"
+               izz="0.10" />
+    </inertial>
       <inertia ixx="8.7002718e-03" ixy="-4.7576583e-05" ixz="1.1160499e-04"
                iyy="8.6195418e-03" iyz="-3.5422299e-06"
                izz="1.4612727e-02" />
     </inertial>
+      -->
   </link>
   <joint name="wheel_left_joint" type="continuous">
-    <parent link="base_link"/>
+    <parent link="differential_link"/>
     <child link="wheel_left_link"/>
-    <origin xyz="${base_offset_x} ${base_offset_y} ${base_offset_z}" rpy="0 0 0"/>
+    <origin xyz="0.20 0.185 0" rpy="0 0 0"/>
+    <axis xyz="0 -1 0"/>
+  </joint>
+  <link name="wheel_left_link">
+    <visual>
+      <origin xyz="0 0 0" rpy="0 0 0"/>
+      <geometry>
+        <mesh filename="package://handirob_description/meshes/wheels/wheel_only.stl" scale="0.001 0.001 0.001"/>
+      </geometry>
+      <material name="dark"/>
+    </visual>
+    <collision>
+      <origin xyz="0 0.0125 0" rpy="-${pi_half} ${pi_half/2} 0"/>
+      <geometry>
+        <cylinder length="0.018" radius="0.085"/>
+      </geometry>
+    </collision>
+    <inertial>
+      <origin xyz="0 0.0125 0" />
+      <mass value="0.338959" />
+      <inertia ixx="0.008" ixy="0.0" ixz="0.0"
+               iyy="0.008" iyz="0.0"
+               izz="0.014365" />
+      </inertial>
+  </link>
+  <joint name="wheel_right_joint" type="continuous">
+    <parent link="differential_link"/>
+    <child link="wheel_right_link"/>
+    <origin xyz="0.20 -0.185 0" rpy="0 0 0"/>
     <axis xyz="0 1 0"/>
   </joint>
-  <link name="wheel_left_link">
-    <visual>
+  <link name="wheel_right_link">
+    <visual>
+      <origin xyz="0 0 0" rpy="${pi} 0 0"/>
+      <geometry>
+        <mesh filename="package://handirob_description/meshes/wheels/wheel_only.stl" scale="0.001 0.001 0.001"/>
+      </geometry>
+      <material name="dark"/>
+    </visual>
+    <collision>
+      <origin xyz="0 -0.0125 0" rpy="${pi_half} ${pi_half/2} 0"/>
+      <geometry>
+        <cylinder length="0.018" radius="0.085"/>
+      </geometry>
+    </collision>
+    <inertial>
+      <origin xyz="0 -0.0125 0" />
+      <mass value="0.338959" />
+      <inertia ixx="0.008" ixy="0.0" ixz="0.0"
+               iyy="0.008" iyz="0.0"
+               izz="0.014365" />
+      </inertial>
+  </link>
+  <joint name="caster_back_right_joint" type="fixed">
+    <parent link="differential_link"/>
+    <child link="caster_back_right_link"/>
+    <origin xyz="-0.220 -0.210 -0.041" rpy="0 0 0"/>
+  </joint>
+  <link name="caster_back_right_link">
+    <collision>
       <origin xyz="0 0 0" rpy="0 0 0"/>
       <geometry>
-        <mesh filename="package://handirob_description/meshes/wheels/wheel_only.stl" scale="0.001 0.001 0.001"/>
-      </geometry>
-      <material name="dark"/>
-    </visual>
-    <collision>
-      <origin xyz="0 0.0125 0" rpy="${pi_half} 0 0"/>
-      <geometry>
-        <cylinder length="0.025" radius="0.0845"/>
-      </geometry>
-    </collision>
-    <inertial>
-      <origin xyz="0 0 0" />
-      <mass value="0.338959" />
-      <inertia ixx="1.1175580e-05" ixy="-4.2369783e-11" ixz="-5.9381719e-09"
-               iyy="1.1192413e-05" iyz="-1.4400107e-11"
-               izz="2.0712558e-05" />
-      </inertial>
-  </link>
-  <joint name="wheel_right_joint" type="continuous">
-    <parent link="base_link"/>
-    <child link="wheel_right_link"/>
-    <origin xyz="${base_offset_x} -${base_offset_y} ${base_offset_z}" rpy="0 0 0"/>
-    <axis xyz="0 1 0"/>
-  </joint>
-  <link name="wheel_right_link">
-    <visual>
-      <origin xyz="0 0 0" rpy="${pi} 0 0"/>
-      <geometry>
-        <mesh filename="package://handirob_description/meshes/wheels/wheel_only.stl" scale="0.001 0.001 0.001"/>
-      </geometry>
-      <material name="dark"/>
-    </visual>
-    <collision>
-      <origin xyz="0 -0.0125 0" rpy="-${pi_half} 0 0"/>
-      <geometry>
-        <cylinder length="0.025" radius="0.0845"/>
-      </geometry>
-    </collision>
-    <inertial>
-      <origin xyz="0 0 0" />
-      <mass value="0.338959" />
-      <inertia ixx="1.1175580e-05" ixy="-4.2369783e-11" ixz="-5.9381719e-09"
-               iyy="1.1192413e-05" iyz="-1.4400107e-11"
-               izz="2.0712558e-05" />
-      </inertial>
-  </link>
-  <joint name="caster_back_right_joint" type="fixed">
-    <parent link="base_link"/>
-    <child link="caster_back_right_link"/>
-    <origin xyz="-0.2 -0.21 0" rpy="0 0 0"/>
-  </joint>
-  <link name="caster_back_right_link">
+        <sphere radius="0.05"/>
+      </geometry>
+    </collision>
+    <inertial>
+      <origin xyz="0 0 0" />
+      <mass value="0.5" />
+      <inertia ixx="0.001" ixy="0.0" ixz="0.0"
+               iyy="0.001" iyz="0.0"
+               izz="0.001" />
+    </inertial>
+  </link>
+  <joint name="caster_back_left_joint" type="fixed">
+    <parent link="differential_link"/>
+    <child link="caster_back_left_link"/>
+    <origin xyz="-0.220 0.21 -0.041" rpy="0 0 0"/>
+  </joint>
+  <link name="caster_back_left_link">
     <collision>
       <origin xyz="0 0 0" rpy="0 0 0"/>
       <geometry>
-        <sphere radius="0.032"/>
-      </geometry>
-    </collision>
-    <inertial>
-      <origin xyz="0 0 0" />
-      <mass value="0.005" />
-      <inertia ixx="0.001" ixy="0.0" ixz="0.0"
-               iyy="0.001" iyz="0.0"
-               izz="0.001" />
-    </inertial>
-  </link>
-  <joint name="caster_back_left_joint" type="fixed">
-    <parent link="base_link"/>
-    <child link="caster_back_left_link"/>
-    <origin xyz="-0.2 0.21 0" rpy="0 0 0"/>
-  </joint>
-  <link name="caster_back_left_link">
-    <collision>
-      <origin xyz="0 0 0" rpy="0 0 0"/>
-      <geometry>
-        <sphere radius="0.032"/>
-      </geometry>
-    </collision>
-    <inertial>
-      <origin xyz="0 0 0" />
-      <mass value="0.005" />
+        <sphere radius="0.05"/>
+      </geometry>
+    </collision>
+    <inertial>
+      <origin xyz="0 0 0" />
+      <mass value="0.5" />
       <inertia ixx="0.001" ixy="0.0" ixz="0.0"
                iyy="0.001" iyz="0.0"
@@ -134,26 +147,26 @@
   </link>
   <joint name="imu_joint" type="fixed">
-    <parent link="base_link"/>
+    <parent link="differential_link"/>
     <child link="imu_link"/>
-    <origin xyz="0.185 -0.048 0.145" rpy="0 0 ${pi}"/>
+    <origin xyz="0.185 -0.048 0.145" rpy="0 0 0"/>
   </joint>
   <link name="imu_link"/>
   <joint name="scan_joint_right" type="fixed">
-    <parent link="base_link"/>
+    <parent link="differential_link"/>
     <child link="right_scan"/>
-    <origin xyz="0.101374 -0.157273 0.268" rpy="0 0 ${pi}"/>
+    <origin xyz="0.115 -0.15 0.21" rpy="0 0 ${pi}"/>
   </joint>
   <link name="right_scan">
     <visual>
-      <origin xyz="0 0 0" rpy="0 0 0"/>
-      <geometry>
-        <mesh filename="package://handirob_description/meshes/sensors/lds.stl" scale="0.001 0.001 0.001"/>
-      </geometry>
-      <material name="dark"/>
-    </visual>
-    <collision>
-      <origin xyz="0 0 0" rpy="0 0 0"/>
-      <geometry>
-        <cylinder length="0.0315" radius="0.055"/>
+      <origin xyz="0.03 0 0" rpy="0 0 ${pi}"/>
+      <geometry>
+        <mesh filename="package://handirob_description/meshes/sensors/RP-lidar-A1v2.stl" scale="0.001 0.001 0.001"/>
+      </geometry>
+      <material name="dark"/>
+    </visual>
+    <collision>
+      <origin xyz="0.03 0 0.025" rpy="0 0 0"/>
+      <geometry>
+        <cylinder length="0.02" radius="0.035"/>
       </geometry>
     </collision>
@@ -167,20 +180,20 @@
   </link>
   <joint name="scan_joint_left" type="fixed">
-    <parent link="base_link"/>
+    <parent link="differential_link"/>
     <child link="left_scan"/>
-    <origin xyz="0.101374 0.157273 0.268" rpy="0 0 ${pi}"/>
+    <origin xyz="0.115 0.15 0.21" rpy="0 0 ${pi}"/>
   </joint>
   <link name="left_scan">
     <visual>
-      <origin xyz="0 0 0" rpy="0 0 0"/>
-      <geometry>
-        <mesh filename="package://handirob_description/meshes/sensors/lds.stl" scale="0.001 0.001 0.001"/>
-      </geometry>
-      <material name="dark"/>
-    </visual>
-    <collision>
-      <origin xyz="0 0 0" rpy="0 0 0"/>
-      <geometry>
-        <cylinder length="0.0315" radius="0.055"/>
+      <origin xyz="0.03 0 0" rpy="0 0 ${pi}"/>
+      <geometry>
+        <mesh filename="package://handirob_description/meshes/sensors/RP-lidar-A1v2.stl" scale="0.001 0.001 0.001"/>
+      </geometry>
+      <material name="dark"/>
+    </visual>
+    <collision>
+      <origin xyz="0.03 0 0.025" rpy="0 0 0"/>
+      <geometry>
+        <cylinder length="0.02" radius="0.035"/>
       </geometry>
     </collision>
@@ -193,6 +206,6 @@
     </inertial>
   </link>
-<xacro:sensor_d435 parent="base_link" use_nominal_extrinsics="false" add_plug="false" use_mesh="true">
-  <origin xyz="0.215 0.016 0.18" rpy="0 -0.6 0"/>
+<xacro:sensor_d435 parent="differential_link" use_nominal_extrinsics="false" add_plug="false" use_mesh="true">
+  <origin xyz="0.205 0 0.18" rpy="0 0 0"/>
 </xacro:sensor_d435>
 </robot>
